File: darwin-radio.sch (EAGLE design)
At the start: 40 parts, among them Q2 NDS8434, U1 ATWINC, U6 MCP7384X

Commit message: Fixed Wifi enable, Radio Pullups, BAT+ connection on charger, and internal layer shorts to various vias.
Parts:
- removed U$10: M55-6102042R, Conservify:M55-6102042R
- removed U$8, U$9: 505110-1692, Conservify:505110-1692
- added J1, J2: 505110-1692, Conservify:505110-1692
- added J3: M55-6102042R, Conservify:M55-6102042R
- added R6, R7: 100k, SparkFun-Resistors:100KOHM-0603-1/10W-1%
Connections:
- net 3V3: now also J3.PIN11, J3.PIN12, R6.2, R7.2; no longer U$10.PIN11, U$10.PIN12
- net BAT+: now also U6.VBAT
- net GND: now also J1.P1, J1.P2, J1.P3, J1.P4, J2.P1, J2.P2, J2.P3, J2.P4, J3.PIN19, J3.PIN20; no longer U$10.PIN19, U$10.PIN20, U$8.P1, U$8.P2, U$8.P3, U$8.P4, U$9.P1, U$9.P2, U$9.P3, U$9.P4
- net MOD_G0: now also J1.P13, J2.P13; no longer U$8.P13, U$9.P13
- net MOD_G1: now also J3.PIN1; no longer U$10.PIN1
- net MOD_G13: now also J1.P14, J2.P14; no longer U$8.P14, U$9.P14
- net MOD_G14: now also J1.P12, J2.P12; no longer U$8.P12, U$9.P12
- net MOD_G2: now also J3.PIN2; no longer U$10.PIN2
- net MOD_G3: now also J3.PIN3; no longer U$10.PIN3
- net MOD_G4: now also J3.PIN4; no longer U$10.PIN4
- net MOD_G5: now also J3.PIN5; no longer U$10.PIN5
- net MOD_MISO: now also J3.PIN10; no longer U$10.PIN10
- net MOD_MOSI: now also J3.PIN8; no longer U$10.PIN8
- net MOD_SCK: now also J3.PIN9; no longer U$10.PIN9
- net MOD_SCL: now also J3.PIN6; no longer U$10.PIN6
- net MOD_SDA: now also J3.PIN7; no longer U$10.PIN7
- net N$17: no longer U6.VBAT
- net RADIO_MISO: now also J1.P9, J2.P9; no longer U$8.P9, U$9.P9
- net RADIO_MOSI: now also J1.P10, J2.P10; no longer U$8.P10, U$9.P10
- net RADIO_SCK: now also J1.P11, J2.P11; no longer U$8.P11, U$9.P11
- net RAD_SCL: now also J1.P16, J2.P16, R6.1; no longer U$8.P16, U$9.P16
- net RAD_SDA: now also J1.P15, J2.P15, R7.1; no longer U$8.P15, U$9.P15
- net UNREG: now also J1.P5, J1.P6, J1.P7, J1.P8, J2.P5, J2.P6, J2.P7, J2.P8, J3.PIN13, J3.PIN14; no longer U$10.PIN13, U$10.PIN14, U$8.P5, U$8.P6, U$8.P7, U$8.P8, U$9.P5, U$9.P6, U$9.P7, U$9.P8
- net WIFI_3V3: now also U1.ENABLE
- net WIFI_CS: now also U1.SSN; no longer U1.ENABLE
- net XX1: now also J3.PIN18; no longer U$10.PIN18
- net XX2: now also J3.PIN17; no longer U$10.PIN17
- net XX3: now also J3.PIN16; no longer U$10.PIN16
- net XX4: now also J3.PIN15; no longer U$10.PIN15
Other:
- note added: "GPS"
- note added: "WIFI"
- moved on the sheet: C11, C12, C2, C4, C5, C7, C8, C9, CBAT1, CREG1, D1, D3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

Commit message: Added external button header. added mounting point for single 'backpack' module. Panelized. PA1.
Parts:
- added FID1, FID2, FID3, FID4: FIDUCIAL_1MM, microbuilder:FIDUCIAL_1MM
- added R8: 100k, SparkFun-Resistors:100KOHM-0603-1/10W-1%
- added U$8: 2X6-HEADERSDS, Conservify:2X6-HEADERSDS
- added U$9: B2B-PH-SM4-TB, Conservify:B2B-PH-SM4-TB
Connections:
- net MOD_G12 renamed CHARGING
- net MOD_G3 renamed HOTSWAP_INT
- net MOD_G6 renamed GPS_ENABLE
- net MOD_G7 renamed WIFI_ENABLE
- removed net MOD_G1: J3.PIN1, LOWER1.PIN2
- removed net MOD_G4: J3.PIN4, LOWER1.PIN17
- removed net X1: UPPER1.PIN3
- new net BACKPACK_ENABLE: U$8.PIN4, UPPER1.PIN3
- new net EEPROM_PROT: J3.PIN1, LOWER1.PIN2, U$8.PIN5
- new net PIN7: U$8.PIN7
- new net XBTN: J3.PIN4, LOWER1.PIN17, R8.2, U$9.P$2
- net 3V3: now also R8.1, U$8.PIN3
- net GND: now also U$8.PIN2, U$9.P$1
- net MOD_G2: now also U$8.PIN6
- net MOD_MISO: now also U$8.PIN10
- net MOD_MOSI: now also U$8.PIN11
- net MOD_SCK: now also U$8.PIN12
- net MOD_SCL: now also U$8.PIN8
- net MOD_SDA: now also U$8.PIN9
- net UNREG: now also U$8.PIN1
Changed lines of the file:
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@@
 <part name="R6" library="SparkFun-Resistors" library_urn="urn:adsk.eagle:library:532" deviceset="100KOHM" device="-0603-1/10W-1%" package3d_urn="urn:adsk.eagle:package:39650/1" value="100k"/>
 <part name="R7" library="SparkFun-Resistors" library_urn="urn:adsk.eagle:library:532" deviceset="100KOHM" device="-0603-1/10W-1%" package3d_urn="urn:adsk.eagle:package:39650/1" value="100k"/>
+<part name="U$8" library="Conservify" library_urn="urn:adsk.eagle:library:11839183" deviceset="2X6-HEADERS" device="DS" package3d_urn="urn:adsk.eagle:package:11839231/2"/>
+<part name="FID1" library="microbuilder" deviceset="FIDUCIAL" device="_1MM"/>
+<part name="FID2" library="microbuilder" deviceset="FIDUCIAL" device="_1MM"/>
+<part name="FID3" library="microbuilder" deviceset="FIDUCIAL" device="_1MM"/>
+<part name="FID4" library="microbuilder" deviceset="FIDUCIAL" device="_1MM"/>
+<part name="U$9" library="Conservify" library_urn="urn:adsk.eagle:library:11839183" deviceset="B2B-PH-SM4-TB" device="" package3d_urn="urn:adsk.eagle:package:11839237/2"/>
+<part name="R8" library="SparkFun-Resistors" library_urn="urn:adsk.eagle:library:532" deviceset="100KOHM" device="-0603-1/10W-1%" package3d_urn="urn:adsk.eagle:package:39650/1" value="100k"/>
 </parts>
 <sheets>
@@
 <attribute name="VALUE" x="210.82" y="21.844" size="1.778" layer="96" font="vector" rot="R180" align="top-center"/>
 </instance>
+<instance part="U$8" gate="G$1" x="467.36" y="33.02" smashed="yes">
+<attribute name="NAME" x="457.2" y="43.434" size="1.27" layer="95"/>
+</instance>
+<instance part="FID1" gate="G$1" x="464.82" y="-30.48" smashed="yes"/>
+<instance part="FID2" gate="G$1" x="464.82" y="-35.56" smashed="yes"/>
+<instance part="FID3" gate="G$1" x="464.82" y="-40.64" smashed="yes"/>
+<instance part="FID4" gate="G$1" x="464.82" y="-45.72" smashed="yes"/>
+<instance part="U$9" gate="G$1" x="317.5" y="38.1" smashed="yes">
+<attribute name="NAME" x="312.674" y="43.942" size="1.778" layer="94"/>
+</instance>
+<instance part="R8" gate="G$1" x="325.12" y="27.94" smashed="yes" rot="R180">
+<attribute name="NAME" x="325.12" y="26.416" size="1.778" layer="95" font="vector" rot="R180" align="bottom-center"/>
+<attribute name="VALUE" x="325.12" y="29.464" size="1.778" layer="96" font="vector" rot="R180" align="top-center"/>
+</instance>
 </instances>
 <busses>
@@
 <label x="259.08" y="66.04" size="1.778" layer="95"/>
 </segment>
+<segment>
+<pinref part="U$8" gate="G$1" pin="PIN9"/>
+<wire x1="482.6" y1="30.48" x2="495.3" y2="30.48" width="0.1524" layer="91"/>
+<label x="492.76" y="30.48" size="1.778" layer="95" align="bottom-right"/>
+</segment>
 </net>
 <net name="MOD_SCL" class="0">
@@
 <label x="259.08" y="68.58" size="1.778" layer="95"/>
 </segment>
+<segment>
+<pinref part="U$8" gate="G$1" pin="PIN8"/>
+<wire x1="482.6" y1="27.94" x2="495.3" y2="27.94" width="0.1524" layer="91"/>
+<label x="492.76" y="27.94" size="1.778" layer="95" align="bottom-right"/>
+</segment>
 </net>
 <net name="RAD_SDA" class="0">
@@
 <label x="259.08" y="63.5" size="1.778" layer="95"/>
 </segment>
+<segment>
+<pinref part="U$8" gate="G$1" pin="PIN11"/>
+<wire x1="482.6" y1="35.56" x2="495.3" y2="35.56" width="0.1524" layer="91"/>
+<label x="492.76" y="35.56" size="1.778" layer="95" align="bottom-right"/>
+</segment>
 </net>
 <net name="MOD_SCK" class="0">
@@
 <label x="259.08" y="60.96" size="1.778" layer="95"/>
 </segment>
+<segment>
+<pinref part="U$8" gate="G$1" pin="PIN12"/>
+<wire x1="482.6" y1="38.1" x2="495.3" y2="38.1" width="0.1524" layer="91"/>
+<label x="492.76" y="38.1" size="1.778" layer="95" align="bottom-right"/>
+</segment>
 </net>
 <net name="MOD_MISO" class="0">
@@
 <label x="259.08" y="58.42" size="1.778" layer="95"/>
 </segment>
+<segment>
+<pinref part="U$8" gate="G$1" pin="PIN10"/>
+<wire x1="482.6" y1="33.02" x2="495.3" y2="33.02" width="0.1524" layer="91"/>
+<label x="492.76" y="33.02" size="1.778" layer="95" align="bottom-right"/>
+</segment>
 </net>
 <net name="MOD_G0" class="0">
@@
 </segment>
 </net>
-<net name="MOD_G1" class="0">
+<net name="EEPROM_PROT" class="0">
 <segment>
 <pinref part="LOWER1" gate="G$1" pin="PIN2"/>
@@
 <label x="259.08" y="81.28" size="1.778" layer="95"/>
 </segment>
+<segment>
+<pinref part="U$8" gate="G$1" pin="PIN5"/>
+<wire x1="452.12" y1="27.94" x2="439.42" y2="27.94" width="0.1524" layer="91"/>
+<label x="441.96" y="27.94" size="1.778" layer="95"/>
+</segment>
 </net>
 <net name="MOD_G2" class="0">
@@
 <label x="259.08" y="78.74" size="1.778" layer="95"/>
 </segment>
-</net>
-<net name="MOD_G3" class="0">
+<segment>
+<pinref part="U$8" gate="G$1" pin="PIN6"/>
+<wire x1="452.12" y1="25.4" x2="439.42" y2="25.4" width="0.1524" layer="91"/>
+<label x="441.96" y="25.4" size="1.778" layer="95"/>
+</segment>
+</net>
+<net name="HOTSWAP_INT" class="0">
 <segment>
 <pinref part="LOWER1" gate="G$1" pin="PIN3"/>
@@
 </segment>
 </net>
-<net name="MOD_G4" class="0">
+<net name="XBTN" class="0">
 <segment>
 <pinref part="LOWER1" gate="G$1" pin="PIN17"/>
@@
 <label x="259.08" y="73.66" size="1.778" layer="95"/>
 </segment>
+<segment>
+<pinref part="U$9" gate="G$1" pin="P$2"/>
+<wire x1="320.04" y1="33.02" x2="320.04" y2="27.94" width="0.1524" layer="91"/>
+<label x="322.58" y="20.32" size="1.778" layer="95"/>
+<pinref part="R8" gate="G$1" pin="2"/>
+<wire x1="320.04" y1="27.94" x2="320.04" y2="17.78" width="0.1524" layer="91"/>
+<junction x="320.04" y="27.94"/>
+</segment>
 </net>
 <net name="MOD_G5" class="0">
@@
 </segment>
 </net>
-<net name="MOD_G6" class="0">
+<net name="GPS_ENABLE" class="0">
 <segment>
 <pinref part="LOWER1" gate="G$1" pin="PIN16"/>
@@
 </segment>
 </net>
-<net name="MOD_G7" class="0">
+<net name="WIFI_ENABLE" class="0">
 <segment>
 <pinref part="LOWER1" gate="G$1" pin="PIN5"/>
@@
 <label x="419.1" y="-48.26" size="1.778" layer="95"/>
 </segment>
+<segment>
+<pinref part="U$8" gate="G$1" pin="PIN2"/>
+<wire x1="452.12" y1="35.56" x2="439.42" y2="35.56" width="0.1524" layer="91"/>
+<label x="441.96" y="35.56" size="1.778" layer="95"/>
+</segment>
+<segment>
+<pinref part="U$9" gate="G$1" pin="P$1"/>
+<wire x1="314.96" y1="33.02" x2="314.96" y2="20.32" width="0.1524" layer="91"/>
+<label x="309.88" y="30.48" size="1.778" layer="95"/>
+</segment>
 </net>
 <net name="3V3" class="0">
@@
 <label x="193.04" y="25.4" size="1.778" layer="95"/>
 </segment>
+<segment>
+<pinref part="U$8" gate="G$1" pin="PIN3"/>
+<wire x1="452.12" y1="33.02" x2="439.42" y2="33.02" width="0.1524" layer="91"/>
+<label x="441.96" y="33.02" size="1.778" layer="95"/>
+</segment>
+<segment>
+<pinref part="R8" gate="G$1" pin="1"/>
+<wire x1="330.2" y1="27.94" x2="335.28" y2="27.94" width="0.1524" layer="91"/>
+<label x="330.2" y="27.94" size="1.778" layer="95"/>
+</segment>
 </net>
 <net name="N$10" class="0">
@@
 </segment>
 </net>
-<net name="X1" class="0">
+<net name="BACKPACK_ENABLE" class="0">
 <segment>
 <pinref part="UPPER1" gate="G$1" pin="PIN3"/>
 <wire x1="269.24" y1="119.38" x2="248.92" y2="119.38" width="0.1524" layer="91"/>
 <label x="251.46" y="119.38" size="1.778" layer="95"/>
+</segment>
+<segment>
+<pinref part="U$8" gate="G$1" pin="PIN4"/>
+<wire x1="452.12" y1="30.48" x2="439.42" y2="30.48" width="0.1524" layer="91"/>
+<label x="441.96" y="30.48" size="1.778" layer="95"/>
 </segment>
 </net>
@@
 <label x="342.9" y="121.92" size="1.778" layer="95"/>
 </segment>
+<segment>
+<pinref part="U$8" gate="G$1" pin="PIN1"/>
+<wire x1="452.12" y1="38.1" x2="439.42" y2="38.1" width="0.1524" layer="91"/>
+<label x="441.96" y="38.1" size="1.778" layer="95"/>
+</segment>
 </net>
 <net name="SOL+" class="0">
@@
 </segment>
 </net>
-<net name="MOD_G12" class="0">
+<net name="CHARGING" class="0">
 <segment>
 <pinref part="UPPER1" gate="G$1" pin="PIN9"/>
@@
 </segment>
 </net>
+<net name="PIN7" class="0">
+<segment>
+<pinref part="U$8" gate="G$1" pin="PIN7"/>
+<wire x1="482.6" y1="25.4" x2="495.3" y2="25.4" width="0.1524" layer="91"/>
+<label x="492.76" y="25.4" size="1.778" layer="95" align="bottom-right"/>
+</segment>
+</net>

Commit message: Cleanup.
Parts:
- removed J1, J2: 505110-1692, Conservify:505110-1692
- removed J3: M55-6102042R, Conservify:M55-6102042R
- removed U$6, U$7, U$9: B2B-PH-SM4-TB, Conservify:B2B-PH-SM4-TB
- removed U$8: 2X6-HEADERSDS, Conservify:2X6-HEADERSDS
- added BACKPACK: 2X6-HEADERSDS, Conservify:2X6-HEADERSDS
- added BACKPLANE: M55-6102042R, Conservify:M55-6102042R
- added BAT-JST, BTN-JST, SOLAR-JST: B2B-PH-SM4-TB, Conservify:B2B-PH-SM4-TB
- added FFC1, FFC2: 505110-1692, Conservify:505110-1692
- C3, C4, C8: value (none) -> 470pf
Connections:
- net 3V3: now also BACKPACK.PIN3, BACKPLANE.PIN11, BACKPLANE.PIN12; no longer J3.PIN11, J3.PIN12, U$8.PIN3
- net BACKPACK_ENABLE: now also BACKPACK.PIN4; no longer U$8.PIN4
- net BAT+: now also BAT-JST.P$1; no longer U$7.P$1
- net BAT-: now also BAT-JST.P$2; no longer U$7.P$2
- net EEPROM_PROT: now also BACKPACK.PIN5, BACKPLANE.PIN1; no longer J3.PIN1, U$8.PIN5
- net GND: now also BACKPACK.PIN2, BACKPLANE.PIN19, BACKPLANE.PIN20, BTN-JST.P$1, FFC1.P1, FFC1.P2, FFC1.P3, FFC1.P4, FFC2.P1, FFC2.P2, FFC2.P3, FFC2.P4, SOLAR-JST.P$2; no longer J1.P1, J1.P2, J1.P3, J1.P4, J2.P1, J2.P2, J2.P3, J2.P4, J3.PIN19, J3.PIN20, U$6.P$2, U$8.PIN2, U$9.P$1
- net HOTSWAP_INT: now also BACKPLANE.PIN3; no longer J3.PIN3
- net MOD_G0: now also FFC1.P13, FFC2.P13; no longer J1.P13, J2.P13
- net MOD_G13: now also FFC1.P14, FFC2.P14; no longer J1.P14, J2.P14
- net MOD_G14: now also FFC1.P12, FFC2.P12; no longer J1.P12, J2.P12
- net MOD_G2: now also BACKPACK.PIN6, BACKPLANE.PIN2; no longer J3.PIN2, U$8.PIN6
- net MOD_G5: now also BACKPLANE.PIN5; no longer J3.PIN5
- net MOD_MISO: now also BACKPACK.PIN10, BACKPLANE.PIN10; no longer J3.PIN10, U$8.PIN10
- net MOD_MOSI: now also BACKPACK.PIN11, BACKPLANE.PIN8; no longer J3.PIN8, U$8.PIN11
- net MOD_SCK: now also BACKPACK.PIN12, BACKPLANE.PIN9; no longer J3.PIN9, U$8.PIN12
- net MOD_SCL: now also BACKPACK.PIN8, BACKPLANE.PIN6; no longer J3.PIN6, U$8.PIN8
- net MOD_SDA: now also BACKPACK.PIN9, BACKPLANE.PIN7; no longer J3.PIN7, U$8.PIN9
- net PIN7: now also BACKPACK.PIN7; no longer U$8.PIN7
- net RADIO_MISO: now also FFC1.P9, FFC2.P9; no longer J1.P9, J2.P9
- net RADIO_MOSI: now also FFC1.P10, FFC2.P10; no longer J1.P10, J2.P10
- net RADIO_SCK: now also FFC1.P11, FFC2.P11; no longer J1.P11, J2.P11
- net RAD_SCL: now also FFC1.P16, FFC2.P16; no longer J1.P16, J2.P16
- net RAD_SDA: now also FFC1.P15, FFC2.P15; no longer J1.P15, J2.P15
- net SOL+: now also SOLAR-JST.P$1; no longer U$6.P$1
- net UNREG: now also BACKPACK.PIN1, BACKPLANE.PIN13, BACKPLANE.PIN14, FFC1.P5, FFC1.P6, FFC1.P7, FFC1.P8, FFC2.P5, FFC2.P6, FFC2.P7, FFC2.P8; no longer J1.P5, J1.P6, J1.P7, J1.P8, J2.P5, J2.P6, J2.P7, J2.P8, J3.PIN13, J3.PIN14, U$8.PIN1
- net XBTN: now also BACKPLANE.PIN4, BTN-JST.P$2; no longer J3.PIN4, U$9.P$2
- net XX1: now also BACKPLANE.PIN18; no longer J3.PIN18
- net XX2: now also BACKPLANE.PIN17; no longer J3.PIN17
- net XX3: now also BACKPLANE.PIN16; no longer J3.PIN16
- net XX4: now also BACKPLANE.PIN15; no longer J3.PIN15
Other:
- note added: "I2C TERM"
- moved on the sheet: C1, C11, C12, C2, C3, C4, C5, C6, CBAT1, CREG1, D1, D3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

Commit message: Added solar pre-regulation, deprecated fuel gauge, added current sense, replaced current sense resistors, lots of routing changes, new panel.
Parts:
- removed CBAT1: 0.1uF, SparkFun-Capacitors:0.1UF-0603-25V-(+80/-20%)
- removed CREG1: 10uF, SparkFun-Capacitors:10UF-0603-6.3V-20%
- removed FID1, FID2, FID3, FID4: FIDUCIAL_1MM, microbuilder:FIDUCIAL_1MM
- removed RSENSE3: 100M, SparkFun-Resistors:1MOHM-0603-1/4W-5%
- removed U$12: MAX17055, Conservify:MAX17055
- added C10, C13: 22uf, rcl:C-USC0603K
- added J1: S1911-46R, Conservify:S1911-46R
- added R10, R9: 100k, SparkFun-Resistors:100KOHM-0603-1/10W-1%
- added REG1: V78E06-1000-SMT-TR, Conservify:V78E06-1000-SMT-TR
- added RX2: 100M, rcl:R-US_R2512
- added U2: INA219, Conservify:INA219
- RX1: device SparkFun-Resistors:1MOHM-0603-1/4W-5% -> rcl:R-US_R2512
Connections:
- removed net BAT-: BAT-JST.P$2, CBAT1.2, CREG1.2, RSENSE3.1, U$12.CSP, U$12.PAD
- removed net N$19: CREG1.1, U$12.REG
- new net BAT+RAW: BAT-JST.P$1, RX2.2, U2.IN+
- new net SOLREG: C13.1, D3.ANODE2, J1.P$1, REG1.VOUT
- net 3V3: now also R10.2, R9.2, U2.VCC
- net BAT+: now also RX2.1, U2.IN-; no longer BAT-JST.P$1, CBAT1.1, U$12.BATT
- net GND: now also BAT-JST.P$2, C10.2, C13.2, REG1.GND, U1.PAD, U2.AD0, U2.AD1, U2.GND; no longer RSENSE3.2, U$12.CSN
- net MOD_SCL: now also R9.1, U2.SCL
- net MOD_SDA: now also R10.1, U2.SDA
- net RAD_SCL: no longer U$12.SCL
- net RAD_SDA: no longer U$12.SDA
- net SOL+: now also C10.1, J1.P$2, REG1.EN, REG1.VIN; no longer D3.ANODE2

Commit message: Added power switch headers.
Parts:
- added J2: (no value), SparkFun-Connectors:CONN_02LOCK_LONGPADS
Connections:
- removed net N$8: R1.2, U$4.EN, U$5.2
- new net PSWITCH: J2.1, R1.2, U$4.EN, U$5.2
- net UNREG: now also J2.2
Changed lines of the file:
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@@
 <?xml version="1.0" encoding="utf-8"?>
 <!DOCTYPE eagle SYSTEM "eagle.dtd">
-<eagle version="9.5.0">
+<eagle version="9.5.2">
 <drawing>
 <settings>
-<setting alwaysvectorfont="yes"/>
+<setting alwaysvectorfont="no"/>
 <setting verticaltext="up"/>
 </settings>
@@
 <part name="C10" library="rcl" library_urn="urn:adsk.eagle:library:334" deviceset="C-US" device="C0603K" package3d_urn="urn:adsk.eagle:package:23680/2" value="22uf"/>
 <part name="C13" library="rcl" library_urn="urn:adsk.eagle:library:334" deviceset="C-US" device="C0603K" package3d_urn="urn:adsk.eagle:package:23680/2" value="22uf"/>
+<part name="J2" library="SparkFun-Connectors" library_urn="urn:adsk.eagle:library:513" deviceset="CONN_02" device="LOCK_LONGPADS" package3d_urn="urn:adsk.eagle:package:38047/1"/>
 </parts>
 <sheets>
@@
 <attribute name="VALUE" x="529.336" y="-27.051" size="1.778" layer="96"/>
 </instance>
+<instance part="J2" gate="G$1" x="187.96" y="35.56" smashed="yes">
+<attribute name="VALUE" x="185.42" y="30.734" size="1.778" layer="96" font="vector"/>
+<attribute name="NAME" x="185.42" y="41.148" size="1.778" layer="95" font="vector"/>
+</instance>
 </instances>
 <busses>
@@
 </segment>
 </net>
-<net name="N$8" class="0">
+<net name="PSWITCH" class="0">
 <segment>
 <pinref part="U$5" gate="G$1" pin="2"/>
@@
 <wire x1="190.5" y1="-2.54" x2="190.5" y2="0" width="0.1524" layer="91"/>
 <junction x="190.5" y="0"/>
+<label x="191.008" y="-2.286" size="1.778" layer="95"/>
+</segment>
+<segment>
+<pinref part="J2" gate="G$1" pin="1"/>
+<wire x1="195.58" y1="35.56" x2="205.74" y2="35.56" width="0.1524" layer="91"/>
+<label x="195.58" y="35.56" size="1.778" layer="95"/>
 </segment>
 </net>
@@
 <label x="254" y="50.8" size="1.778" layer="95"/>
 </segment>
-</net>
+<segment>
+<pinref part="J2" gate="G$1" pin="2"/>
+<wire x1="195.58" y1="38.1" x2="205.74" y2="38.1" width="0.1524" layer="91"/>
+<label x="195.58" y="38.1" size="1.778" layer="95"/>
+</segment>
+</net>
